Commit message: nero_pipeline: collect the lab's final launch scripts, configuration and environment snapshot (2026-10-14)

File: nero_pipeline/config_snapshots/agx_arm_moveit/agx_arm.srdf.xacro (robot description, xacro)
@@ -373,4 +373,13 @@
       <joint name="joint7" value="0.040317105721069016" />
     </group_state>
+    <group_state name="initial" group="arm">
+      <joint name="joint1" value="1.7453292519943296e-05" />
+      <joint name="joint2" value="-1.043968692080408" />
+      <joint name="joint3" value="-5.235987755982989e-05" />
+      <joint name="joint4" value="2.08" />
+      <joint name="joint5" value="6.981317007977319e-05" />
+      <joint name="joint6" value="0.002513274122871835" />
+      <joint name="joint7" value="0.43399357180090997" />
+    </group_state>
 </xacro:if>
   <!-- ======================== ARM DISABLE COLLISIONS ======================== -->
